Commit message: Full model

File: examples/multibody/BarrettHand/models/BarrettFinger.xacro (robot description, xacro)
@@ -18,4 +18,5 @@
       <xacro:property name="j" value="-1" />
     </xacro:if>
+    <!-- DH Parameters -->
     <xacro:property name="A0" value="${0.025 * r}"/>
     <xacro:property name="A1" value="0.05"/>
@@ -26,5 +27,5 @@
     <xacro:property name="alpha2" value="0"/>
     <xacro:property name="alpha3" value="-1.5707963"/>
-    <xacro:property name="D0" value="0.0589"/>
+    <xacro:property name="D0" value="0.0589"/>  <!-- Offset determined from the CAD -->
     <xacro:property name="D1" value="0"/>
     <xacro:property name="D2" value="0"/>
@@ -120,5 +121,5 @@
       </visual>
     </link>
-    <frame name="finger_${index}_tip">
+    <frame name="finger_${index}_tip" attached_to="finger_${index}_distal">
       <pose relative_to="finger_${index}_distal">${A3} 0 ${D3} ${alpha3} 0 ${theta3}</pose>
     </frame>
@@ -138,6 +139,6 @@
         <xyz>0 0 ${r}</xyz>
 	      <limit>
-	        <lower>-inf</lower>
-	        <upper>inf</upper>
+	        <lower>0</lower>
+	        <upper>3.141592653589793</upper>
           <effort>0</effort>
         </limit>
@@ -152,6 +153,6 @@
         <xyz>0 0 1</xyz>
 	      <limit>
-	        <lower>-inf</lower>
-	        <upper>inf</upper>
+	        <lower>0</lower>
+	        <upper>2.443460952792061</upper>
           <effort>0</effort>
         </limit>
@@ -165,6 +166,6 @@
         <xyz>0 0 1</xyz>
 	      <limit>
-	        <lower>-inf</lower>
-	        <upper>inf</upper>
+	        <lower>0</lower>
+	        <upper>0.8377580409572781</upper>
           <effort>0</effort>
         </limit>
